File: PCB/HX711_LOADCELL_AMP.sch (KiCad schematic (older format))
At the start: 21 parts

Commit message: complete loadcell connector
Parts:
- J?: symbol Connector:Conn_01x04_Female -> Connector:Conn_01x05_Female
Connections:
- net GND: now also J?.5 (Pin_5)
- net A-: now reaches J?.4 (Pin_4), R?.2
- net A+: now reaches J?.3 (Pin_3), R?.2
Other:
- note added: "RED\nBLACK\nGREEN/BLUE\nWHITE\nYELLOW"
Changed lines of the file:
@@
 E+
 $Comp
-L Connector:Conn_01x04_Female J?
+L Connector:Conn_01x05_Female J?
 U 1 1 5E8B3AD7
-P 4100 5350
-F 0 "J?" H 4128 5326 50  0000 L CNN
-F 1 "LOADCELL" H 4128 5235 50  0000 L CNN
-F 2 "" H 4100 5350 50  0001 C CNN
-F 3 "~" H 4100 5350 50  0001 C CNN
-	1    4100 5350
+P 4100 5450
+F 0 "J?" H 3950 5150 50  0000 L CNN
+F 1 "LOADCELL" H 3800 5050 50  0000 L CNN
+F 2 "" H 4100 5450 50  0001 C CNN
+F 3 "~" H 4100 5450 50  0001 C CNN
+	1    4100 5450
 	-1   0    0    -1
 $EndComp
@@
 L power:GND #PWR?
 U 1 1 5E8B6772
-P 4350 5350
-F 0 "#PWR?" H 4350 5100 50  0001 C CNN
-F 1 "GND" V 4355 5222 50  0000 R CNN
-F 2 "" H 4350 5350 50  0001 C CNN
-F 3 "" H 4350 5350 50  0001 C CNN
-	1    4350 5350
+P 4400 5350
+F 0 "#PWR?" H 4400 5100 50  0001 C CNN
+F 1 "GND" V 4405 5222 50  0000 R CNN
+F 2 "" H 4400 5350 50  0001 C CNN
+F 3 "" H 4400 5350 50  0001 C CNN
+	1    4400 5350
 	0    -1   -1   0
 $EndComp
 Wire Wire Line
-	4350 5350 4300 5350
+	4400 5350 4300 5350
 Wire Wire Line
 	4850 5350 4700 5350
@@
 	0    1    1    0
 $EndComp
+$Comp
+L power:GND #PWR?
+U 1 1 5E8E0E20
+P 4400 5650
+F 0 "#PWR?" H 4400 5400 50  0001 C CNN
+F 1 "GND" V 4405 5522 50  0000 R CNN
+F 2 "" H 4400 5650 50  0001 C CNN
+F 3 "" H 4400 5650 50  0001 C CNN
+	1    4400 5650
+	0    -1   -1   0
+$EndComp
+Wire Wire Line
+	4400 5650 4300 5650
+Text Label 4300 5450 0    50   ~ 0
+A+
+Text Label 4300 5550 0    50   ~ 0
+A-
+Text Label 4300 5350 0    50   ~ 0
+E-
+Text Label 4300 5650 0    50   ~ 0
+SH
+Text Notes 4050 5700 2    63   ~ 0
+RED\nBLACK\nGREEN/BLUE\nWHITE\nYELLOW
 $EndSCHEMATC
