File: PCB/ENDSTOP.sch (KiCad schematic (older format))
At the start: 4 parts

Commit message: Annotated Schematic
Parts:
- gave numbers to parts that had none: 4
Changed lines of the file:
@@
 OUTPUT
 $Comp
-L Switch:SW_SPST SW?
+L Switch:SW_SPST SW3
 U 1 1 5E8A8DC4
 P 6150 4150
-F 0 "SW?" V 6104 4248 50  0000 L CNN
+F 0 "SW3" V 6104 4248 50  0000 L CNN
 F 1 "ENDSTOP" V 6195 4248 50  0000 L CNN
 F 2 "" H 6150 4150 50  0001 C CNN
-F 3 "~" H 6150 4150 50  0001 C CNN
+F 3 "" H 6150 4150 50  0001 C CNN
 	1    6150 4150
 	0    1    1    0
 $EndComp
 $Comp
-L Device:C_Small C?
+L Device:C_Small C44
 U 1 1 5E8A9073
 P 5900 4150
-F 0 "C?" H 5809 4196 50  0000 R CNN
+F 0 "C44" H 5809 4196 50  0000 R CNN
 F 1 "100nF" H 5809 4105 50  0000 R CNN
 F 2 "" H 5900 4150 50  0001 C CNN
-F 3 "~" H 5900 4150 50  0001 C CNN
+F 3 "" H 5900 4150 50  0001 C CNN
 	1    5900 4150
 	1    0    0    -1
 $EndComp
 $Comp
-L Device:R_Small R?
+L Device:R_Small R24
 U 1 1 5E8A974E
 P 6150 3750
-F 0 "R?" H 6209 3796 50  0000 L CNN
+F 0 "R24" H 6209 3796 50  0000 L CNN
 F 1 "10k" H 6209 3705 50  0000 L CNN
 F 2 "" H 6150 3750 50  0001 C CNN
-F 3 "~" H 6150 3750 50  0001 C CNN
+F 3 "" H 6150 3750 50  0001 C CNN
 	1    6150 3750
 	1    0    0    -1
@@
 	6150 3900 6150 3950
 $Comp
-L power:GND #PWR?
+L power:GND #PWR0122
 U 1 1 5E8A9B1B
 P 5900 4400
-F 0 "#PWR?" H 5900 4150 50  0001 C CNN
+F 0 "#PWR0122" H 5900 4150 50  0001 C CNN
 F 1 "GND" H 5905 4227 50  0000 C CNN
 F 2 "" H 5900 4400 50  0001 C CNN
@@
 $EndComp
 $Comp
-L power:GND #PWR?
+L power:GND #PWR0124
 U 1 1 5E8A9B96
 P 6150 4400
-F 0 "#PWR?" H 6150 4150 50  0001 C CNN
+F 0 "#PWR0124" H 6150 4150 50  0001 C CNN
 F 1 "GND" H 6155 4227 50  0000 C CNN
 F 2 "" H 6150 4400 50  0001 C CNN
@@
 	5900 4400 5900 4250
 $Comp
-L power:+3.3V #PWR?
+L power:+3.3V #PWR0123
 U 1 1 5E8AA8C2
 P 6150 3600
-F 0 "#PWR?" H 6150 3450 50  0001 C CNN
+F 0 "#PWR0123" H 6150 3450 50  0001 C CNN
 F 1 "+3.3V" H 6165 3773 50  0000 C CNN
 F 2 "" H 6150 3600 50  0001 C CNN
@@
 	7000 3900 6650 3900
 $Comp
-L Connector:Conn_01x02_Female J?
+L Connector:Conn_01x02_Female J9
 U 1 1 5E8ACECE
 P 6900 4100
-F 0 "J?" H 6928 4076 50  0000 L CNN
+F 0 "J9" H 6928 4076 50  0000 L CNN
 F 1 "ENDSTOP_CONN" H 6928 3985 50  0000 L CNN
 F 2 "" H 6900 4100 50  0001 C CNN
-F 3 "~" H 6900 4100 50  0001 C CNN
+F 3 "" H 6900 4100 50  0001 C CNN
 	1    6900 4100
 	1    0    0    -1
@@
 	6650 3900 6150 3900
 $Comp
-L power:GND #PWR?
+L power:GND #PWR0125
 U 1 1 5E8AD764
 P 6650 4400
-F 0 "#PWR?" H 6650 4150 50  0001 C CNN
+F 0 "#PWR0125" H 6650 4150 50  0001 C CNN
 F 1 "GND" H 6655 4227 50  0000 C CNN
 F 2 "" H 6650 4400 50  0001 C CNN

Commit message: Added Dielectric and voltage rating to all capacitors
Parts:
- C44: Dielectric (none) -> X7R; Voltage Rating (none) -> 6.3V
Changed lines of the file:
@@
 $Descr A4 11693 8268
 encoding utf-8
-Sheet 14 20
+Sheet 16 20
 Title ""
 Date ""
@@
 F 2 "" H 5900 4150 50  0001 C CNN
 F 3 "" H 5900 4150 50  0001 C CNN
+F 4 "X7R" H 5900 4150 50  0001 C CNN "Dielectric"
+F 5 "6.3V" H 5900 4150 50  0001 C CNN "Voltage Rating"
 	1    5900 4150
 	1    0    0    -1
