File: PCB/POWER_SUPPLY.sch (KiCad schematic (older format))
At the start: 12 parts

Commit message: Annotated Schematic
Parts:
- gave numbers to parts that had none: 12
Changed lines of the file:
@@
 $EndDescr
 $Comp
-L Device:Battery BT?
+L Device:Battery BT1
 U 1 1 5E90B731
 P 5600 3650
-F 0 "BT?" H 5708 3696 50  0000 L CNN
+F 0 "BT1" H 5708 3696 50  0000 L CNN
 F 1 "LEAD_ACID" H 5708 3605 50  0000 L CNN
 F 2 "" V 5600 3710 50  0001 C CNN
-F 3 "~" V 5600 3710 50  0001 C CNN
+F 3 "" V 5600 3710 50  0001 C CNN
 	1    5600 3650
 	1    0    0    -1
@@
 	5600 3200 5600 3450
 $Comp
-L power:GND #PWR?
+L power:GND #PWR066
 U 1 1 5E929E4E
 P 5600 3900
-F 0 "#PWR?" H 5600 3650 50  0001 C CNN
+F 0 "#PWR066" H 5600 3650 50  0001 C CNN
 F 1 "GND" H 5605 3727 50  0000 C CNN
 F 2 "" H 5600 3900 50  0001 C CNN
@@
 Connection ~ 3950 2800
 $Comp
-L power:GND #PWR?
+L power:GND #PWR064
 U 1 1 5E92F162
 P 3800 3050
-F 0 "#PWR?" H 3800 2800 50  0001 C CNN
+F 0 "#PWR064" H 3800 2800 50  0001 C CNN
 F 1 "GND" H 3805 2877 50  0000 C CNN
 F 2 "" H 3800 3050 50  0001 C CNN
@@
 	6100 2800 6100 3200
 $Comp
-L Converter_ACDC:IRM-20-15 PS?
+L Converter_ACDC:IRM-20-15 PS1
 U 1 1 5E92C858
 P 3350 2900
-F 0 "PS?" H 3350 3225 50  0000 C CNN
+F 0 "PS1" H 3350 3225 50  0000 C CNN
 F 1 "IRM-30-15" H 3350 3134 50  0000 C CNN
 F 2 "" H 3350 2600 50  0001 C CNN
@@
 	6000 3200 6100 3200
 $Comp
-L Device:D_Schottky D?
+L Device:D_Schottky D1
 U 1 1 5E96E6B3
 P 5850 2800
-F 0 "D?" H 5850 2584 50  0000 C CNN
+F 0 "D1" H 5850 2584 50  0000 C CNN
 F 1 "SK34BTR" H 5850 2675 50  0000 C CNN
 F 2 "" H 5850 2800 50  0001 C CNN
@@
 VBATT_SENSE
 $Comp
-L Device:R_Small R?
+L Device:R_Small R11
 U 1 1 5E987A48
 P 5300 3750
-F 0 "R?" H 5359 3796 50  0000 L CNN
+F 0 "R11" H 5359 3796 50  0000 L CNN
 F 1 "10k" H 5359 3705 50  0000 L CNN
 F 2 "" H 5300 3750 50  0001 C CNN
-F 3 "~" H 5300 3750 50  0001 C CNN
+F 3 "" H 5300 3750 50  0001 C CNN
 	1    5300 3750
 	1    0    0    -1
@@
 Connection ~ 5300 3600
 $Comp
-L power:GND #PWR?
+L power:GND #PWR065
 U 1 1 5E989430
 P 5300 3900
-F 0 "#PWR?" H 5300 3650 50  0001 C CNN
+F 0 "#PWR065" H 5300 3650 50  0001 C CNN
 F 1 "GND" H 5305 3727 50  0000 C CNN
 F 2 "" H 5300 3900 50  0001 C CNN
@@
 	5300 3850 5300 3900
 $Comp
-L Device:R_Small R?
+L Device:R_Small R10
 U 1 1 5E98794C
 P 5300 3450
-F 0 "R?" H 5359 3496 50  0000 L CNN
+F 0 "R10" H 5359 3496 50  0000 L CNN
 F 1 "56k" H 5359 3405 50  0000 L CNN
 F 2 "" H 5300 3450 50  0001 C CNN
-F 3 "~" H 5300 3450 50  0001 C CNN
+F 3 "" H 5300 3450 50  0001 C CNN
 	1    5300 3450
 	1    0    0    -1
@@
 	3950 2800 5700 2800
 $Comp
-L Device:D_Schottky D?
+L Device:D_Schottky D2
 U 1 1 5E99D1CB
 P 5850 3200
-F 0 "D?" H 5850 2984 50  0000 C CNN
+F 0 "D2" H 5850 2984 50  0000 C CNN
 F 1 "SK34BTR" H 5850 3075 50  0000 C CNN
 F 2 "" H 5850 3200 50  0001 C CNN
@@
 Connection ~ 6100 2800
 $Comp
-L Device:LED D?
+L Device:LED D3
 U 1 1 5E8B2580
 P 8200 2800
-F 0 "D?" V 8239 2683 50  0000 R CNN
+F 0 "D3" V 8239 2683 50  0000 R CNN
 F 1 "3V3" V 8148 2683 50  0000 R CNN
 F 2 "" H 8200 2800 50  0001 C CNN
-F 3 "~" H 8200 2800 50  0001 C CNN
+F 3 "" H 8200 2800 50  0001 C CNN
 	1    8200 2800
 	0    -1   -1   0
 $EndComp
 $Comp
-L Device:R_Small R?
+L Device:R_Small R12
 U 1 1 5E8B32F4
 P 8200 2500
-F 0 "R?" H 8259 2546 50  0000 L CNN
+F 0 "R12" H 8259 2546 50  0000 L CNN
 F 1 "1k" H 8259 2455 50  0000 L CNN
 F 2 "" H 8200 2500 50  0001 C CNN
-F 3 "~" H 8200 2500 50  0001 C CNN
+F 3 "" H 8200 2500 50  0001 C CNN
 	1    8200 2500
 	1    0    0    -1
@@
 	8200 2600 8200 2650
 $Comp
-L power:GND #PWR?
+L power:GND #PWR067
 U 1 1 5E8B38F1
 P 8200 3000
-F 0 "#PWR?" H 8200 2750 50  0001 C CNN
+F 0 "#PWR067" H 8200 2750 50  0001 C CNN
 F 1 "GND" H 8205 2827 50  0000 C CNN
 F 2 "" H 8200 3000 50  0001 C CNN
@@
 	8200 2950 8200 3000
 $Comp
-L Device:LED D?
+L Device:LED D4
 U 1 1 5E8B5AE6
 P 8550 2800
-F 0 "D?" V 8589 2683 50  0000 R CNN
+F 0 "D4" V 8589 2683 50  0000 R CNN
 F 1 "12V" V 8498 2683 50  0000 R CNN
 F 2 "" H 8550 2800 50  0001 C CNN
-F 3 "~" H 8550 2800 50  0001 C CNN
+F 3 "" H 8550 2800 50  0001 C CNN
 	1    8550 2800
 	0    -1   -1   0
 $EndComp
 $Comp
-L Device:R_Small R?
+L Device:R_Small R13
 U 1 1 5E8B5AEC
 P 8550 2500
-F 0 "R?" H 8609 2546 50  0000 L CNN
+F 0 "R13" H 8609 2546 50  0000 L CNN
 F 1 "1k" H 8609 2455 50  0000 L CNN
 F 2 "" H 8550 2500 50  0001 C CNN
-F 3 "~" H 8550 2500 50  0001 C CNN
+F 3 "" H 8550 2500 50  0001 C CNN
 	1    8550 2500
 	1    0    0    -1
@@
 	8550 2600 8550 2650
 $Comp
-L power:GND #PWR?
+L power:GND #PWR068
 U 1 1 5E8B5AF3
 P 8550 3000
-F 0 "#PWR?" H 8550 2750 50  0001 C CNN
+F 0 "#PWR068" H 8550 2750 50  0001 C CNN
 F 1 "GND" H 8555 2827 50  0000 C CNN
 F 2 "" H 8550 3000 50  0001 C CNN
@@
 	6100 3200 6200 3200
 $Comp
-L Device:LED D?
+L Device:LED D5
 U 1 1 5E8B6ACE
 P 8900 2800
-F 0 "D?" V 8939 2683 50  0000 R CNN
+F 0 "D5" V 8939 2683 50  0000 R CNN
 F 1 "15V" V 8848 2683 50  0000 R CNN
 F 2 "" H 8900 2800 50  0001 C CNN
-F 3 "~" H 8900 2800 50  0001 C CNN
+F 3 "" H 8900 2800 50  0001 C CNN
 	1    8900 2800
 	0    -1   -1   0
 $EndComp
 $Comp
-L Device:R_Small R?
+L Device:R_Small R14
 U 1 1 5E8B6AD4
 P 8900 2500
-F 0 "R?" H 8959 2546 50  0000 L CNN
+F 0 "R14" H 8959 2546 50  0000 L CNN
 F 1 "1k" H 8959 2455 50  0000 L CNN
 F 2 "" H 8900 2500 50  0001 C CNN
-F 3 "~" H 8900 2500 50  0001 C CNN
+F 3 "" H 8900 2500 50  0001 C CNN
 	1    8900 2500
 	1    0    0    -1
@@
 	8900 2600 8900 2650
 $Comp
-L power:GND #PWR?
+L power:GND #PWR069
 U 1 1 5E8B6ADB
 P 8900 3000
-F 0 "#PWR?" H 8900 2750 50  0001 C CNN
+F 0 "#PWR069" H 8900 2750 50  0001 C CNN
 F 1 "GND" H 8905 2827 50  0000 C CNN
 F 2 "" H 8900 3000 50  0001 C CNN

Commit message: Added some footprints
Parts:
- PS1: footprint (none) -> custom:IRM-30-xx
Changed lines of the file:
@@
 F 0 "PS1" H 3350 3225 50  0000 C CNN
 F 1 "IRM-30-15" H 3350 3134 50  0000 C CNN
-F 2 "" H 3350 2600 50  0001 C CNN
+F 2 "custom:IRM-30-xx" H 3350 2600 50  0001 C CNN
 F 3 "https://www.meanwell.com/Upload/PDF/IRM-30/IRM-30-SPEC.PDF" H 3750 2550 50  0001 C CNN
 	1    3350 2900
