File: PCB/SSD1306_OLED.sch (KiCad schematic (older format))
At the start: 1 part

Commit message: Annotated Schematic
Parts:
- gave numbers to parts that had none: 1
Changed lines of the file:
@@
 $EndDescr
 $Comp
-L Connector:Conn_01x04_Female J?
+L Connector:Conn_01x04_Female J5
 U 1 1 5E8F6533
 P 5850 4050
-F 0 "J?" H 5878 4026 50  0000 L CNN
+F 0 "J5" H 5878 4026 50  0000 L CNN
 F 1 "OLED_I2C" H 5878 3935 50  0000 L CNN
 F 2 "" H 5850 4050 50  0001 C CNN
-F 3 "~" H 5850 4050 50  0001 C CNN
+F 3 "" H 5850 4050 50  0001 C CNN
 	1    5850 4050
 	1    0    0    -1
 $EndComp
 $Comp
-L power:GND #PWR?
+L power:GND #PWR054
 U 1 1 5E86600D
 P 5600 3950
-F 0 "#PWR?" H 5600 3700 50  0001 C CNN
+F 0 "#PWR054" H 5600 3700 50  0001 C CNN
 F 1 "GND" V 5605 3822 50  0000 R CNN
 F 2 "" H 5600 3950 50  0001 C CNN
@@
 	5600 3950 5650 3950
 $Comp
-L power:+3.3V #PWR?
+L power:+3.3V #PWR055
 U 1 1 5E86671F
 P 5600 4050
-F 0 "#PWR?" H 5600 3900 50  0001 C CNN
+F 0 "#PWR055" H 5600 3900 50  0001 C CNN
 F 1 "+3.3V" V 5615 4178 50  0000 L CNN
 F 2 "" H 5600 4050 50  0001 C CNN
