File: PCB/AIR_HUMIDITY_SENSOR.sch (KiCad schematic (older format))
At the start: 0 parts

Commit message: Added Humidity and temperature sensors
Parts:
- added C49: 220nF, symbol Device:C_Small
- added U11: HIH712x, symbol custom:HIH712x
Connections:
- new net +5V: C49.1, U11.1 (VDD)
- new net GND: C49.2, U11.2 (VSS)
- new net SCL: U11.3 (SCL)
- new net SDA: U11.4 (SDA)
Changed lines of the file:
@@
 Comment4 ""
 $EndDescr
+$Comp
+L custom:HIH712x U11
+U 1 1 5E9303FE
+P 5800 3900
+F 0 "U11" H 6250 4250 50  0000 R CNN
+F 1 "HIH712x" H 5950 3900 50  0000 R CNN
+F 2 "" H 5800 3900 50  0001 C CNN
+F 3 "" H 5800 3900 50  0001 C CNN
+	1    5800 3900
+	1    0    0    -1
+$EndComp
+$Comp
+L Device:C_Small C49
+U 1 1 5E931061
+P 5950 2850
+F 0 "C49" H 6042 2896 50  0000 L CNN
+F 1 "220nF" H 6042 2805 50  0000 L CNN
+F 2 "" H 5950 2850 50  0001 C CNN
+F 3 "~" H 5950 2850 50  0001 C CNN
+F 4 "X7R" H 5950 2850 50  0001 C CNN "Dielectric"
+F 5 "6.3V" H 5950 2850 50  0001 C CNN "Voltage Rating"
+	1    5950 2850
+	1    0    0    -1
+$EndComp
+$Comp
+L power:+5V #PWR0159
+U 1 1 5E93133D
+P 5950 2700
+F 0 "#PWR0159" H 5950 2550 50  0001 C CNN
+F 1 "+5V" H 5965 2873 50  0000 C CNN
+F 2 "" H 5950 2700 50  0001 C CNN
+F 3 "" H 5950 2700 50  0001 C CNN
+	1    5950 2700
+	1    0    0    -1
+$EndComp
+$Comp
+L power:GND #PWR0158
+U 1 1 5E93145F
+P 5800 4350
+F 0 "#PWR0158" H 5800 4100 50  0001 C CNN
+F 1 "GND" H 5805 4177 50  0000 C CNN
+F 2 "" H 5800 4350 50  0001 C CNN
+F 3 "" H 5800 4350 50  0001 C CNN
+	1    5800 4350
+	1    0    0    -1
+$EndComp
+$Comp
+L power:+5V #PWR0157
+U 1 1 5E93181D
+P 5800 3450
+F 0 "#PWR0157" H 5800 3300 50  0001 C CNN
+F 1 "+5V" H 5815 3623 50  0000 C CNN
+F 2 "" H 5800 3450 50  0001 C CNN
+F 3 "" H 5800 3450 50  0001 C CNN
+	1    5800 3450
+	1    0    0    -1
+$EndComp
+$Comp
+L power:GND #PWR0160
+U 1 1 5E931D8D
+P 5950 3000
+F 0 "#PWR0160" H 5950 2750 50  0001 C CNN
+F 1 "GND" H 5955 2827 50  0000 C CNN
+F 2 "" H 5950 3000 50  0001 C CNN
+F 3 "" H 5950 3000 50  0001 C CNN
+	1    5950 3000
+	1    0    0    -1
+$EndComp
+Wire Wire Line
+	5950 2700 5950 2750
+Wire Wire Line
+	5800 3450 5800 3500
+Wire Wire Line
+	5950 2950 5950 3000
+Wire Wire Line
+	5800 4300 5800 4350
+Text HLabel 6350 3850 2    50   BiDi ~ 0
+SDA
+Text HLabel 6350 3950 2    50   Input ~ 0
+SCL
 $EndSCHEMATC
