File: PCB/FAN_CONTROLLER.sch (KiCad schematic (older format))
At the start: 3 parts, among them J11 FAN, Q4 MMBT4401-7-F

Commit message: Roughly connected nets
Changed lines of the file:
@@
 Wire Wire Line
 	6100 4350 6100 4400
-Text HLabel 5550 4150 0    50   Input ~ 0
+Text HLabel 5500 4150 0    50   Input ~ 0
 CTRL
+Wire Wire Line
+	5500 4150 5550 4150
 $EndSCHEMATC
