File: PCB/DIFFERENTIAL_PRESSURE.sch (KiCad schematic (older format))
At the start: 5 parts, among them U16 MPXV7002

Commit message: Added differential pressure sensor MPN
Parts:
- U16: MPN (none) -> MPXV7002DP
Changed lines of the file:
@@
 F 2 "custom:MPXV7002" H 5550 3500 50  0001 C CNN
 F 3 "https://www.nxp.com/docs/en/data-sheet/MPXV7002.pdf" H 6050 4450 50  0001 C CNN
+F 4 "MPXV7002DP" H 6050 3850 50  0001 C CNN "MPN"
 	1    6050 3850
 	1    0    0    -1
