File: PCB/TFT_DISPLAY.sch (KiCad schematic (older format))
At the start: 16 parts, among them Q5 MMBT4401-7-F, U17 62684-45110E9ALF, U18 74LVC245, U19 74LVC245, U21 DT024CTFT(-TS)

Commit message: Added some footprints
Parts:
- C50, C51, C52, C53: footprint (none) -> Capacitor_SMD:C_0603_1608Metric; Dielectric (none) -> X7R; Voltage Rating (none) -> 6.3V
- R44, R45, R46: footprint (none) -> Resistor_SMD:R_0603_1608Metric
- TP24, TP6, TP7, TP8: footprint (none) -> custom:TestPoint_Pad_D1.5mm
- U18, U19: footprint (none) -> Package_SO:TSSOP-20_4.4x6.5mm_P0.65mm
Changed lines of the file:
@@
 F 0 "R44" V 8054 4700 50  0000 C CNN
 F 1 "1k" V 8145 4700 50  0000 C CNN
-F 2 "" H 8250 4700 50  0001 C CNN
+F 2 "Resistor_SMD:R_0603_1608Metric" H 8250 4700 50  0001 C CNN
 F 3 "~" H 8250 4700 50  0001 C CNN
 	1    8250 4700
@@
 F 0 "R46" V 7154 4350 50  0000 C CNN
 F 1 "120R" V 7245 4350 50  0000 C CNN
-F 2 "" H 7350 4350 50  0001 C CNN
+F 2 "Resistor_SMD:R_0603_1608Metric" H 7350 4350 50  0001 C CNN
 F 3 "~" H 7350 4350 50  0001 C CNN
 F 4 "1/4W" V 7350 4350 50  0001 C CNN "Power Rating"
@@
 F 0 "U18" H 2800 3250 50  0000 C CNN
 F 1 "74LVC245" H 3300 1950 50  0000 C CNN
-F 2 "" H 3050 2600 50  0001 C CNN
+F 2 "Package_SO:TSSOP-20_4.4x6.5mm_P0.65mm" H 3050 2600 50  0001 C CNN
 F 3 "http://www.ti.com/lit/ds/symlink/sn74lvc245a.pdf" H 3050 2600 50  0001 C CNN
 	1    3050 2600
@@
 F 0 "R45" H 1891 5204 50  0000 R CNN
 F 1 "10k" H 1891 5295 50  0000 R CNN
-F 2 "" H 1950 5250 50  0001 C CNN
+F 2 "Resistor_SMD:R_0603_1608Metric" H 1950 5250 50  0001 C CNN
 F 3 "~" H 1950 5250 50  0001 C CNN
 	1    1950 5250
@@
 F 0 "C50" H 2942 1346 50  0000 L CNN
 F 1 "100nF" H 2942 1255 50  0000 L CNN
-F 2 "" H 2850 1300 50  0001 C CNN
+F 2 "Capacitor_SMD:C_0603_1608Metric" H 2850 1300 50  0001 C CNN
 F 3 "~" H 2850 1300 50  0001 C CNN
+F 4 "X7R" H 2850 1300 50  0001 C CNN "Dielectric"
+F 5 "6.3V" H 2850 1300 50  0001 C CNN "Voltage Rating"
 	1    2850 1300
 	1    0    0    -1
@@
 F 0 "C51" H 3392 1346 50  0000 L CNN
 F 1 "100nF" H 3392 1255 50  0000 L CNN
-F 2 "" H 3300 1300 50  0001 C CNN
+F 2 "Capacitor_SMD:C_0603_1608Metric" H 3300 1300 50  0001 C CNN
 F 3 "~" H 3300 1300 50  0001 C CNN
+F 4 "X7R" H 3300 1300 50  0001 C CNN "Dielectric"
+F 5 "6.3V" H 3300 1300 50  0001 C CNN "Voltage Rating"
 	1    3300 1300
 	1    0    0    -1
@@
 F 0 "C52" H 6142 2196 50  0000 L CNN
 F 1 "100nF" H 6142 2105 50  0000 L CNN
-F 2 "" H 6050 2150 50  0001 C CNN
+F 2 "Capacitor_SMD:C_0603_1608Metric" H 6050 2150 50  0001 C CNN
 F 3 "~" H 6050 2150 50  0001 C CNN
+F 4 "X7R" H 6050 2150 50  0001 C CNN "Dielectric"
+F 5 "6.3V" H 6050 2150 50  0001 C CNN "Voltage Rating"
 	1    6050 2150
 	1    0    0    -1
@@
 F 0 "C53" H 6592 2196 50  0000 L CNN
 F 1 "10uF" H 6592 2105 50  0000 L CNN
-F 2 "" H 6500 2150 50  0001 C CNN
+F 2 "Capacitor_SMD:C_0603_1608Metric" H 6500 2150 50  0001 C CNN
 F 3 "~" H 6500 2150 50  0001 C CNN
+F 4 "X7R" H 6500 2150 50  0001 C CNN "Dielectric"
+F 5 "6.3V" H 6500 2150 50  0001 C CNN "Voltage Rating"
 	1    6500 2150
 	1    0    0    -1
@@
 F 0 "U19" H 2800 5350 50  0000 C CNN
 F 1 "74LVC245" H 3300 4050 50  0000 C CNN
-F 2 "" H 3050 4700 50  0001 C CNN
+F 2 "Package_SO:TSSOP-20_4.4x6.5mm_P0.65mm" H 3050 4700 50  0001 C CNN
 F 3 "http://www.ti.com/lit/ds/symlink/sn74lvc245a.pdf" H 3050 4700 50  0001 C CNN
 	1    3050 4700
@@
 F 0 "TP7" V 6654 5788 50  0000 L CNN
 F 1 "XR" V 6745 5788 50  0000 L CNN
-F 2 "" H 6900 5600 50  0001 C CNN
+F 2 "custom:TestPoint_Pad_D1.5mm" H 6900 5600 50  0001 C CNN
 F 3 "~" H 6900 5600 50  0001 C CNN
 	1    6700 5600
@@
 F 0 "TP6" V 6654 5588 50  0000 L CNN
 F 1 "XL" V 6745 5588 50  0000 L CNN
-F 2 "" H 6900 5400 50  0001 C CNN
+F 2 "custom:TestPoint_Pad_D1.5mm" H 6900 5400 50  0001 C CNN
 F 3 "~" H 6900 5400 50  0001 C CNN
 	1    6700 5400
@@
 F 0 "TP8" V 6654 5988 50  0000 L CNN
 F 1 "YU" V 6745 5988 50  0000 L CNN
-F 2 "" H 6900 5800 50  0001 C CNN
+F 2 "custom:TestPoint_Pad_D1.5mm" H 6900 5800 50  0001 C CNN
 F 3 "~" H 6900 5800 50  0001 C CNN
 	1    6700 5800
@@
 F 0 "TP24" V 6654 6188 50  0000 L CNN
 F 1 "YD" V 6745 6188 50  0000 L CNN
-F 2 "" H 6900 6000 50  0001 C CNN
+F 2 "custom:TestPoint_Pad_D1.5mm" H 6900 6000 50  0001 C CNN
 F 3 "~" H 6900 6000 50  0001 C CNN
 	1    6700 6000
